Commit message: 更新urdf以及拉取libxr

File: src/mysystem/urdf/robot.urdf (robot description, URDF)
Before this commit: robot robot, 6 links, 5 joints
Links:
- added link imu, mass 0.55271082; collision mesh filename=package://mysystem/meshes/imu.stl; visual mesh filename=package://mysystem/meshes/imu.stl
- added link livox_frame, mass 0.33968131; collision mesh filename=package://mysystem/meshes/livox_frame.stl; visual mesh filename=package://mysystem/meshes/livox_frame.stl
- link up: mass 2.83205162 -> 1.9396595
Joints:
- removed joint up_joint
- removed joint wheel_joint_1
- removed joint wheel_joint_2
- removed joint wheel_joint_3
- removed joint wheel_joint_4
- added joint joint_imu: type fixed, parent up, child imu, origin xyz=0.0768 0.025 0.063 rpy=0 0 0, axis 0 0 1
- added joint joint_livox_frame: type fixed, parent up, child livox_frame, origin xyz=-0.0808 0 0.0951 rpy=0.00000735 0.78539265 3.14159265, axis 0 0 1
- added joint joint_up: type continuous, parent base_link, child up, origin xyz=0 0 0.1039 rpy=0 0 0, axis 0 0 1
- added joint joint_wheel_1: type continuous, parent base_link, child wheel_1, origin xyz=0.11 0.1605 0.0762 rpy=-1.5708 0 0, axis 0 0 1
- added joint joint_wheel_2: type continuous, parent base_link, child wheel_2, origin xyz=-0.11 0.1605 0.0762 rpy=-1.5708 0 0, axis 0 0 1
- added joint joint_wheel_3: type continuous, parent base_link, child wheel_3, origin xyz=-0.11 -0.1605 0.0762 rpy=1.5708 0 0, axis 0 0 1
- added joint joint_wheel_4: type continuous, parent base_link, child wheel_4, origin xyz=0.11 -0.1605 0.0762 rpy=1.5708 0 0, axis 0 0 1

Commit message: 添加控制节点，启动文件

File: src/mysystem/urdf/robot.urdf (robot description, URDF)
Before this commit: robot robot, 8 links, 7 joints
Joints:
- removed joint joint_imu
- added joint joint_imu_up: type fixed, parent imu, child up, origin xyz=-0.0768 -0.025 -0.063 rpy=0 0 0, axis 0 0 1
- joint joint_up: child up -> base_link; origin xyz=0 0 0.1039 rpy=0 0 0 -> xyz=0 0 -0.1039 rpy=0 0 0; parent base_link -> up

Commit message: 看起来能用

File: src/mysystem/urdf/robot.urdf (robot description, URDF)
Before this commit: robot robot, 8 links, 7 joints
Links:
- link wheel_1: geometry collision sphere radius=0.07618; visual mesh filename=package://mysystem/meshes/wheel_1.stl
- link wheel_2: geometry collision sphere radius=0.07618; visual mesh filename=package://mysystem/meshes/wheel_2.stl
- link wheel_3: geometry collision sphere radius=0.07618; visual mesh filename=package://mysystem/meshes/wheel_3.stl
- link wheel_4: geometry collision sphere radius=0.07618; visual mesh filename=package://mysystem/meshes/wheel_4.stl
Joints:
- joint joint_up: type continuous -> fixed
- joint joint_wheel_3: axis 0 0 1 -> 0 0 -1
- joint joint_wheel_4: axis 0 0 1 -> 0 0 -1

Commit message: 加入nav2_params

File: src/mysystem/urdf/robot.urdf (robot description, URDF)
Before this commit: robot robot, 8 links, 7 joints
Links:
- removed link imu
- removed link livox_frame
- added link body, mass 0.33968131; collision mesh filename=package://mysystem/meshes/livox_frame.stl; visual mesh filename=package://mysystem/meshes/livox_frame.stl
Joints:
- removed joint joint_imu_up
- removed joint joint_livox_frame
- added joint joint_body: type fixed, parent body, child up, origin xyz=0.0101109412 -0.0000009142 -0.1243801386 rpy=0.0000103944 0.78539265 -3.1415853037, axis 0 0 1

Commit message: 更改nav2_params，获得map

File: src/mysystem/urdf/robot.urdf (robot description, URDF)
Before this commit: robot robot, 7 links, 6 joints
Links:
- removed link body
- added link aft_mapped, mass 0.33968131; collision mesh filename=package://mysystem/meshes/livox_frame.stl; visual mesh filename=package://mysystem/meshes/livox_frame.stl
Joints:
- removed joint joint_body
- added joint joint_aft_mapped: type fixed, parent aft_mapped, child up, origin xyz=0.0101109412 -0.0000009142 -0.1243801386 rpy=0.0000103944 0.78539265 -3.1415853037, axis 0 0 1

Commit message: 修改nav2_params

File: src/mysystem/urdf/robot.urdf (robot description, URDF)
Before this commit: robot robot, 7 links, 6 joints
Joints:
- joint joint_up: origin xyz=0 0 -0.1039 rpy=0 0 0 -> xyz=0 0 -0.1039 rpy=0 0 3.141592653589793
